File: HARDWARE/ETH1HMSR-SMS/Power.kicad_sch (KiCad schematic)
At the start: 18 parts, among them J201 1715721, Q201 SI5618A, Q202 MMBT3904, U201 TSR_1-2450, U202 TLV62568DBV

Commit message: Development
Other:
- moved on the sheet: C201, C202, C203, C204, C205, D201, D202, F201, J201, Q202, R201, U202
