File: HARDWARE/ETH1HMSR-SMS/ETH1HMSR-SMS.kicad_pcb (KiCad board)
At the start: 2 copper layers, 100 x 45 mm, 112 parts, among them J201 1715721, J301 RJ45_Wuerth_7499010121A, J401 20021111-00010T4LF, J501 1710072, Q201 SI5618A, Q202 MMBT3904, U201 TSR_1-2450, U202 TLV62568DBV, U301 LAN8742A, U401 STM32H743VITx, U402 24LC08B-E/MS, U501 HMSR-SMS, U502 DG419LDY, U503 DG411LEDQ, U504 OPA341UA, U505 OPA341UA, Y301 NX5032GA-25, Y401 NX5032GA-16

Commit message: SW and HW development
Parts:
- added C415: 1u, Capacitor_SMD:C_0603_1608Metric_Pad1.08x0.95mm_HandSolder, F.Cu at (128.2, 94.8)
- added C416: 0.1u, Capacitor_SMD:C_0603_1608Metric_Pad1.08x0.95mm_HandSolder, F.Cu at (128.2, 97.3)
- added C417: 0.1u, Capacitor_SMD:C_0603_1608Metric_Pad1.08x0.95mm_HandSolder, F.Cu at (128.2, 99.8)
- added C418: 1u, Capacitor_SMD:C_0603_1608Metric_Pad1.08x0.95mm_HandSolder, F.Cu at (68.9, 102.0)
- added C509: 0.1u, Capacitor_SMD:C_0603_1608Metric_Pad1.08x0.95mm_HandSolder, F.Cu at (68.9, 79.9)
- added C510: 0.1u, Capacitor_SMD:C_0603_1608Metric_Pad1.08x0.95mm_HandSolder, F.Cu at (68.9, 82.4)
- added C511: 0.1u, Capacitor_SMD:C_0603_1608Metric_Pad1.08x0.95mm_HandSolder, F.Cu at (68.9, 84.9)
- added C512: 0.1u, Capacitor_SMD:C_0603_1608Metric_Pad1.08x0.95mm_HandSolder, F.Cu at (68.9, 87.5)
- added C513: 0.1u, Capacitor_SMD:C_0603_1608Metric_Pad1.08x0.95mm_HandSolder, F.Cu at (68.9, 90.0)
- added C514: 0.1u, Capacitor_SMD:C_0603_1608Metric_Pad1.08x0.95mm_HandSolder, F.Cu at (68.9, 92.5)
- added R407: 0, Resistor_SMD:R_0603_1608Metric_Pad0.98x0.95mm_HandSolder, F.Cu at (128.2, 104.8)
- added R513: RT1206BRE07900KL, Resistor_SMD:R_1206_3216Metric_Pad1.30x1.75mm_HandSolder, F.Cu at (82.5, 93.5)
- added R514: 0, Resistor_SMD:R_0603_1608Metric_Pad0.98x0.95mm_HandSolder, F.Cu at (68.9, 97.5)
- added RN501: SOT-DIV23LF-03-9002-1002-DD, Package_TO_SOT_SMD:SOT-23, F.Cu at (82.2, 80.9)
- added U403: ADR4533, Package_SO:SOIC-8_3.9x4.9mm_P1.27mm, F.Cu at (154.1, 67.8)
- added U506: DG412LEDQ, Package_SO:TSSOP-16_4.4x5mm_P0.65mm, F.Cu at (75.4, 88.5)
- added U507: OPA341UA, Package_SO:SOIC-8_3.9x4.9mm_P1.27mm, F.Cu at (75.3, 95.1)
- R507: value 10k -> 0
- U503: value DG411LEDQ -> DG412LEDQ
- Y401: moved to B.Cu
- moved J401 170.5 mm to (144.7, 95.8), turned to 90 degrees
- moved Y401 165.1 mm to (153.3, 76.5), turned to 180 degrees
- moved R507 150.1 mm to (68.9, 95.0)
- moved U503 48.5 mm to (75.4, 82.0)
- moved U504 7.23 mm to (133.7, 87.5)
- moved U501 0.78 mm to (121.7, 81.9)
- moved J201 0.57 mm to (194.9, 93.6)
- moved U301 0.51 mm to (169.8, 76.1), turned to -90 degrees
- moved J301 0.46 mm to (179.8, 71.8)
- moved U201 0.42 mm to (185.2, 88.0)
Connections:
- R507 pad 1: Net-(R507-Pad1) -> Net-(U504--)
- R507 pad 2: +5VL -> Net-(R507-Pad2)
- R508 pad 1: Net-(U504--) -> Net-(R507-Pad2)
- U401 pad 20: VDDA -> +3.3VADC
- U401 pad 22: /MCU/MCU_DEFAULT -> unconnected-(U401-PA0-Pad22)
- U401 pad 77: unconnected-(U401-PA15-Pad77) -> /MCU/MCU_DEFAULT
- U503 pad 14: Net-(U503-Pad14) -> Net-(R507-Pad2)
- U503 pad 15: Net-(U503-Pad14) -> Net-(U504--)
- U503 pad 16: Net-(R507-Pad1) -> /Current/MCU_MEAS_ENA

Commit message: Updated to Kicad 8
Parts:
- removed R302, R304, R305: 33, Resistor_SMD:R_0603_1608Metric_Pad0.98x0.95mm_HandSolder
- removed R303, R306, R307, R308, R309: 10k, Resistor_SMD:R_0603_1608Metric_Pad0.98x0.95mm_HandSolder
- removed R313, R314, R315, R316: 49R9, Resistor_SMD:R_0603_1608Metric_Pad0.98x0.95mm_HandSolder
- added C515: 100p, Capacitor_SMD:C_0603_1608Metric_Pad1.08x0.95mm_HandSolder, B.Cu at (151.9, 71.4)
- added R515: 100, Resistor_SMD:R_0603_1608Metric_Pad0.98x0.95mm_HandSolder, F.Cu at (151.9, 71.4)
- added RN301: EXB-V8V103JV, Resistor_SMD:R_Array_Concave_4x0603, B.Cu at (164.8, 76.1)
- added RN302: EXB-V8V330JV, Resistor_SMD:R_Array_Concave_4x0603, F.Cu at (164.8, 76.1)
- added RN303: EXB-38V510JV, Resistor_SMD:R_Array_Concave_4x0603, B.Cu at (186.1, 74.9)
- C201, C202, C301, C304, C306, C307, C308, C309, C310, C311, C312, C401, C402, C403, C404, C405, C406, C407, C408, C409, C410, C411, C412, C413, C414, C415, C416, C417, C418, C501, C503, C504, C505, C506, C507, C508, C509, C510, C511, C512, C513, C514, D201, D202, F201, FB401, R202, R311, R312, R317, R318, R401, R402, R403, R404, R405, R407, R501, R502, R503, R504, R505, R506, R507, R510, R511, R512, R513, R514, RN501, U402: moved to B.Cu
- R301: value 33 -> 10k; moved to B.Cu
- moved C311 240.3 mm to (182.2, 69.7), turned to 90 degrees
- moved C312 236.2 mm to (177.5, 75.7), turned to 90 degrees
- moved C307 233.9 mm to (170.9, 82.9), turned to -90 degrees
- moved C310 233.5 mm to (172.5, 82.9), turned to -90 degrees
- moved C304 233.4 mm to (171.3, 69.2), turned to 90 degrees
- moved C309 232.8 mm to (172.1, 78.6), turned to -90 degrees
- moved C308 232.0 mm to (170.7, 72.9), turned to 90 degrees
- moved C302 232.0 mm to (166.5, 83.1), turned to 90 degrees
- moved C305 232.0 mm to (168.0, 83.1), turned to 90 degrees
- moved R311 231.3 mm to (176.9, 83.3), turned to -90 degrees
- moved C301 230.5 mm to (167.3, 69.2), turned to 90 degrees
- moved C303 228.0 mm to (164.8, 73.2), turned to 180 degrees
- moved R317 227.3 mm to (176.9, 79.9), turned to -90 degrees
- moved C306 226.8 mm to (164.8, 73.2), turned to 180 degrees
- moved R318 225.4 mm to (176.9, 69.7), turned to 90 degrees
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Connections:
- D501 pad 3: /Current/HMSR_VOUT -> Net-(D501-K-Pad3)
- R301 pad 1: /Ethernet/MODE0 -> GND
- R301 pad 2: /Ethernet/RMII_RXD0 -> Net-(U301-RXER/PHYAD0)
- R510 pad 1: /Current/HMSR_VOUT -> Net-(D501-K-Pad3)
- R514 pad 2: /Current/HMSR_VOUT -> Net-(D501-K-Pad3)
- U401 pad 18: unconnected-(U401-PC3_C-Pad18) -> /Current/HMSR_VOUT
- U401 pad 37: unconnected-(U401-PE7-Pad37) -> /Current/MCU_G1
- U401 pad 38: unconnected-(U401-PE8-Pad38) -> /Current/MCU_G10
- U401 pad 39: unconnected-(U401-PE9-Pad39) -> /Current/MCU_G100
- U401 pad 40: unconnected-(U401-PE10-Pad40) -> /Current/MCU_DIV1
- U401 pad 41: unconnected-(U401-PE11-Pad41) -> /Current/MCU_DIV10
- U401 pad 42: unconnected-(U401-PE12-Pad42) -> /Current/MCU_DIV100
- U401 pad 43: unconnected-(U401-PE13-Pad43) -> /Current/MCU_MEAS_ENA
- U401 pad 44: unconnected-(U401-PE14-Pad44) -> /Current/MCU_ZOFFS
- U401 pad 45: unconnected-(U401-PE15-Pad45) -> /Current/MCU_DIV_ENA
- U503 pad 3: /Current/HMSR_VOUT -> Net-(D501-K-Pad3)
- U505 pad 6: /Current/HMSR_VOUT -> Net-(D501-K-Pad3)

Commit message: PCB design
Parts:
- C302, C305, D501: moved to B.Cu
- C515: moved to F.Cu
- moved R403 18.3 mm to (164.2, 69.2), turned to -90 degrees
- moved D501 13.1 mm to (141.0, 75.8)
- moved C305 10.2 mm to (168.8, 72.9)
- moved C302 10.2 mm to (167.3, 72.9)
- moved R407 4.26 mm to (155.2, 69.2), turned to -90 degrees
- moved C417 4.08 mm to (151.8, 69.2)
- moved C418 4.08 mm to (153.3, 69.2)
- moved R515 3.18 mm to (154.7, 72.9)
- moved C415 3.05 mm to (158.6, 69.2)
- moved C416 3.05 mm to (157.1, 69.2)
- moved U403 2.92 mm to (155.3, 69.2)
- moved C312 1.89 mm to (176.9, 77.5), turned to 180 degrees
- moved C515 1.61 mm to (151.4, 72.9), turned to 180 degrees
- moved D401 1.28 mm to (139.6, 96.4)
- moved C307 1.02 mm to (169.9, 82.8)
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Connections:
- JP401 pad 1: /MCU/MCU_DEFAULT -> /MCU/MCU_DEF
- R403 pad 1: /MCU/MCU_DEFAULT -> /MCU/MCU_DEF
- U401 pad 1: unconnected-(U401-PE2-Pad1) -> /MCU/MCU_DEF
- U401 pad 77: /MCU/MCU_DEFAULT -> unconnected-(U401-PA15-Pad77)
Routing:
- net +3.3V: track 0.00 -> 77.8 mm, vias 0 -> 23
- net /MCU/NRST: track 0.00 -> 47.1 mm, vias 0 -> 2
- net GND: track 0.00 -> 43.2 mm, vias 0 -> 13
- net Net-(D501-K-Pad3): track 0.00 -> 43.1 mm, vias 0 -> 2
- net +2V5: track 0.00 -> 38.3 mm, vias 0 -> 1
- net /Ethernet/RMII_MDIO: track 0.00 -> 35.3 mm, vias 0 -> 2
- net VCCQ: track 0.00 -> 34.5 mm, vias 0 -> 5
- net Net-(R507-Pad2): track 0.00 -> 31.9 mm, vias 0 -> 1
- net /Ethernet/RMII_CRS_DV: track 0.00 -> 31.0 mm, vias 0 -> 2
- net /Ethernet/RMII_RXD0: track 0.00 -> 30.9 mm, vias 0 -> 2
- net /Ethernet/RMII_TXD1: track 0.00 -> 30.8 mm, vias 0 -> 2
- net /Ethernet/REF_CLK: track 0.00 -> 30.8 mm, vias 0 -> 2
- net /Ethernet/RMII_RXD1: track 0.00 -> 30.7 mm, vias 0 -> 2
- net /Ethernet/RMII_TXEN: track 0.00 -> 30.7 mm, vias 0 -> 2
- net /Ethernet/RMII_TXD0: track 0.00 -> 30.6 mm, vias 0 -> 2
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- added copper zone on B.Cu, net +3.3V
- added copper zone on F.Cu, net +3.3V
- added copper zone on In2.Cu, net +3.3V
- added copper zone on B.Cu, net +5V
- added copper zone on F.Cu, net +5V
- added copper zone on In2.Cu, net +5V
- added copper zone on B.Cu, net +5VL
- added copper zone on F.Cu, net +5VL
- added copper zone on In2.Cu, net +5VL
- added copper zone on B.Cu, net Earth
- added copper zone on F.Cu, net Earth
- added copper zone on B.Cu, net GND
- added copper zone on F.Cu, net GND
- added copper zone on In1.Cu, net GND
- added copper zone on B.Cu, net Net-(J501-Pin_1)
- added copper zone on F.Cu, net Net-(J501-Pin_1)
- added copper zone on In1.Cu, net Net-(J501-Pin_1)
- added copper zone on In2.Cu, net Net-(J501-Pin_1)
- added copper zone on B.Cu, net Net-(J501-Pin_2)
- added copper zone on F.Cu, net Net-(J501-Pin_2)
- added copper zone on In1.Cu, net Net-(J501-Pin_2)
- added copper zone on In2.Cu, net Net-(J501-Pin_2)
- added copper zone on F.Cu, net Net-(U202-SW)
- added copper zone on B.Cu, net VCCQ
- added copper zone on F.Cu, net VCCQ
- added copper zone on In2.Cu, net VCCQ
- added copper zone on B.Cu, net VDDA
Other:
- outline, holes or cut-outs redrawn
- copper layers 2 -> 4

Commit message: Development
Parts:
- moved C411 3.92 mm to (146.7, 90.3), turned to -90 degrees
- moved C201 1.02 mm to (189.2, 87.6)
- moved C202 1.02 mm to (189.2, 90.0)
- moved D201 0.77 mm to (184.8, 96.1)
- moved R202 0.71 mm to (178.1, 90.6)
- moved D202 0.70 mm to (182.4, 90.6)
- moved F201 0.13 mm to (189.5, 95.6)
Connections:
- U401 pad 34: unconnected-(U401-PB0-Pad34) -> /Current/OCD_EXT
- U401 pad 37: /Current/MCU_G1 -> /Current/MCU_G100
- U401 pad 39: /Current/MCU_G100 -> /Current/MCU_MEAS_ENA
- U401 pad 40: /Current/MCU_DIV1 -> /Current/MCU_G1
- U401 pad 43: /Current/MCU_MEAS_ENA -> /Current/MCU_ZOFFS
- U401 pad 44: /Current/MCU_ZOFFS -> /Current/MCU_DIV_ENA
- U401 pad 45: /Current/MCU_DIV_ENA -> /Current/MCU_DIV1
- U401 pad 46: unconnected-(U401-PB10-Pad46) -> /Current/OCD_INT
- U401 pad 63: /MCU/LED_RED -> /MCU/LED_BLUE
- U401 pad 64: /MCU/LED_GREEN -> /MCU/LED_RED
- U401 pad 65: /MCU/LED_BLUE -> /MCU/LED_GREEN
Routing:
- net /Current/MCU_MEAS_ENA: track 2.10 -> 26.3 mm
- net /Current/MCU_G1: track 2.78 -> 25.4 mm
- net /Current/OCD_EXT: track 2.24 -> 24.7 mm, vias 1 -> 2
- net Net-(D201-A): track 3.44 -> 25.4 mm, vias 0 -> 1
- net /Current/MCU_G100: track 2.16 -> 23.8 mm
- net /Current/OCD_INT: track 2.43 -> 22.5 mm, vias 1 -> 2
- net /Current/MCU_DIV1: track 2.56 -> 20.1 mm
- net /Current/MCU_ZOFFS: track 2.86 -> 18.6 mm
- net /Current/MCU_DIV_ENA: track 2.10 -> 17.8 mm
- net /Current/MCU_G10: track 3.05 -> 18.1 mm
- net Net-(D401-RK): track 0.00 -> 14.2 mm
- net Net-(D401-GK): track 1.09 -> 12.4 mm
- net Net-(D202-K): track 0.00 -> 10.5 mm, vias 0 -> 1
- net Net-(D401-BK): track 0.72 -> 8.85 mm
- net +3.3V: track 77.8 -> 85.0 mm, vias 23 -> 25
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- added copper zone on B.Cu, net Net-(D201-K)
- added copper zone on F.Cu, net Net-(D201-K)
- added copper zone on B.Cu, net Net-(J201-Pin_1)
- added copper zone on B.Cu, net Net-(Q201-D)
- added copper zone on F.Cu, net Net-(Q201-D)

Commit message: PCB
Parts:
- U502: value DG419LDY -> DG419LEDY
- moved C501 1.40 mm to (130.0, 96.4)
- moved C502 1.40 mm to (130.0, 96.4)
- moved FB501 1.40 mm to (134.6, 96.4)
- moved D401 1.14 mm to (138.4, 96.4)
- moved C409 0.76 mm to (154.8, 97.2)
- moved J401 0.76 mm to (145.4, 97.8)
- moved R401 0.76 mm to (152.4, 97.2)
Routing:
- net (no net): track 0.00 -> 84.3 mm
- net GND: track 48.6 -> 55.0 mm, vias 23 -> 29
- net +3.3V: track 85.0 -> 79.3 mm
- net Net-(D401-GK): track 12.4 -> 13.7 mm
- net VDDA: track 12.2 -> 10.9 mm
- net Net-(D401-RK): track 14.2 -> 15.3 mm
- net Net-(D401-BK): track 8.85 -> 9.99 mm
- net /MCU/NRST: track 47.1 -> 48.2 mm
- net /MCU/TCK_SWCLK: track 18.2 -> 19.0 mm
- net /MCU/TMS_SWDIO: track 18.0 -> 18.7 mm
Other:
- board text added: "+24 VDC"
- board text added: "1"
- board text added: "2"
- board text added: "3"
- board text added: "4"
- board text added: "ETH1HMSR-SMS Default IP : 196.168.1.17"
- board text added: "HMSR 6-SMS HMSR 8-SMS HMSR 10-SMS HMSR 15-SMS HMSR 20-SMS HMSR 30-SMS"

Commit message: Development
Parts:
- removed R407: 0, Resistor_SMD:R_0603_1608Metric_Pad0.98x0.95mm_HandSolder
- removed the R508 at (134.7, 67.2)
- removed R509: 4k/0.1%, Resistor_SMD:R_0603_1608Metric_Pad0.98x0.95mm_HandSolder
- removed the U403 at (155.3, 69.2)
- added C409: 0.1u, Capacitor_SMD:C_0603_1608Metric_Pad1.08x0.95mm_HandSolder, B.Cu at (157.7, 71.8)
- added C411: 1u, Capacitor_SMD:C_0603_1608Metric_Pad1.08x0.95mm_HandSolder, B.Cu at (156.2, 71.8)
- added C412: 0.1u, Capacitor_SMD:C_0603_1608Metric_Pad1.08x0.95mm_HandSolder, B.Cu at (153.9, 67.1)
- added R406: 0, Resistor_SMD:R_0603_1608Metric_Pad0.98x0.95mm_HandSolder, F.Cu at (150.9, 69.5)
- added RN502: MPMT10012001AT1, Package_TO_SOT_SMD:SOT-23, F.Cu at (135.9, 66.3)
- added U401: LT6350xMS8, Package_SO:MSOP-8_3x3mm_P0.65mm, F.Cu at (154.6, 69.5)
- added U402: REF1933AIDDCT, Package_TO_SOT_SMD:TSOT-23-5_HandSoldering, F.Cu at (159.4, 69.5)
- moved R515 14.3 mm to (142.0, 66.3), turned to 90 degrees
- moved C515 13.5 mm to (139.6, 66.3), turned to -90 degrees
- moved C405 6.35 mm to (157.7, 67.1), turned to 90 degrees
- moved C402 4.38 mm to (162.4, 67.1)
- moved C404 4.38 mm to (160.9, 67.1)
- moved C407 3.63 mm to (156.2, 67.1), turned to 90 degrees
- moved C420 0.25 mm to (150.1, 74.7)
- moved C417 0.25 mm to (150.1, 73.0)
- renumbered C415 to C402, C402 to C403, C416 to C404, C417 to C405, C403 to C406, C418 to C407, C404 to C408, C405 to C410, C406 to C413, C409 to C414, C407 to C415, C408 to C416, C410 to C417, C411 to C418, C413 to C419, C412 to C420, C414 to C421, C511 to C501, C503 to C502, C501 to C503, C512 to C504, C504 to C505, C502 to C506, C513 to C507, C505 to C508, C514 to C509, C509 to C510, C510 to C511, C506 to C512, C507 to C513, C508 to C514, R403 to R401, R401 to R402, R402 to R403, R504 to R501, R501 to R502, R502 to R503, R503 to R504, R513 to R505, R505 to R506, R506 to R507, R507 to R508, R514 to R511, R510 to R512, R511 to R513, R512 to R514, U401 to U403, U402 to U404, U506 to U502, U502 to U503, U503 to U504, U504 to U505, U507 to U506, U505 to U507
Connections:
- R502 pad 1: +2V5 -> +5VL
- R508 pad 2: Net-(R507-Pad2) -> Net-(R508-Pad2)
- R511 pad 1: Net-(U505-+) (its old number) -> Net-(U507-+)
- U403 pad 17: unconnected-(U401-PC2_C-Pad17) -> /MCU/VOUTN
- U403 pad 18: /Current/HMSR_VOUT -> /MCU/VOUTP
- U502 pad 10: +2V5 -> +3.3VADC
- U502 pad 14: Net-(R507-Pad2) -> Net-(U507-+)
- U502 pad 2: +2V5 -> +3.3VADC
- U502 pad 6: +2V5 -> +3.3VADC
- U504 pad 14: Net-(R507-Pad2) -> Net-(R508-Pad2)
- U507 pad 3: Net-(U505-+) (its old number) -> Net-(U507-+)
Routing:
- net +3.3VADC: track 13.1 -> 49.2 mm, vias 1 -> 3
- net +2V5: track 38.2 -> 2.43 mm
- net Net-(R507-Pad2): track 32.2 -> 0.00 mm, vias 1 -> 0
- net Net-(U507-+): track 0.00 -> 24.5 mm, vias 0 -> 1
- net Net-(R508-Pad2): track 0.00 -> 22.9 mm, vias 0 -> 1
- net /MCU/VOUTP: track 0.00 -> 22.0 mm
- net Net-(D501-K-Pad3): track 40.9 -> 21.2 mm
- net Net-(U505-+) (its old number): track 12.8 -> 0.00 mm, vias 1 -> 0
- net /MCU/VOUTN: track 0.00 -> 12.7 mm
- net /Current/HMSR_VOUT: track 4.90 -> 16.1 mm
- net VDDA: track 10.9 -> 1.53 mm
- net +1.65V: track 0.00 -> 7.51 mm, vias 0 -> 2
- net +3.3V: track 79.3 -> 83.9 mm, vias 25 -> 26
- net +5V: track 4.43 -> 8.05 mm
- net +5VL: track 11.5 -> 14.1 mm
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Other:
- board text added: "CURRENT MEASUREMENT"
- board text added: "ETH1HMSR-SMS Default IP : 192.168.1.17"
- board text removed: "ETH1HMSR-SMS Default IP : 196.168.1.17"
- board text removed: "HMSR 6-SMS HMSR 8-SMS HMSR 10-SMS HMSR 15-SMS HMSR 20-SMS HMSR 30-SMS"

Commit message: Development
Parts:
- removed the C509 at (134.1, 92.2)
- removed the C510 at (134.1, 86.4)
- removed the C511 at (141.4, 86.2)
- removed the R505 at (139.7, 92.6)
- removed U505, U506, U507: OPA341UA, Package_SO:SOIC-8_3.9x4.9mm_P1.27mm
- added R407: 0, Resistor_SMD:R_0603_1608Metric_Pad0.98x0.95mm_HandSolder, F.Cu at (151.3, 71.8)
- added R408: 0, Resistor_SMD:R_0603_1608Metric_Pad0.98x0.95mm_HandSolder, F.Cu at (156.0, 71.8)
- added R501: 100k, Resistor_SMD:R_0603_1608Metric_Pad0.98x0.95mm_HandSolder, F.Cu at (137.2, 72.9)
- added R509: 2k5/0.1%, Resistor_SMD:R_0603_1608Metric_Pad0.98x0.95mm_HandSolder, B.Cu at (134.1, 86.9)
- added R510: 2k5/0.1%, Resistor_SMD:R_0603_1608Metric_Pad0.98x0.95mm_HandSolder, B.Cu at (134.1, 91.6)
- added R511: 100k/0.1%, Resistor_SMD:R_0603_1608Metric_Pad0.98x0.95mm_HandSolder, F.Cu at (139.8, 83.9)
- C504, D501, R506: moved to F.Cu
- R507: value 1k -> 1k/0.1%
- R508: value 0 -> 1k/0.1%
- RN501: value SOT-DIV23LF-03-9002-1002-DD -> MPMT10012001AT1; moved to F.Cu
- U502: value DG412LEDQ -> OPA4340UA; footprint Package_SO:TSSOP-16_4.4x5mm_P0.65mm -> Package_SO:SSOP-16_3.9x4.9mm_P0.635mm
- moved RN502 24.2 mm to (133.9, 90.4)
- moved R512 15.5 mm to (140.1, 87.5), turned to 180 degrees
- moved C501 13.4 mm to (134.1, 82.0)
- moved C507 10.3 mm to (138.2, 75.9)
- moved U503 9.88 mm to (140.1, 79.0)
- moved U504 9.65 mm to (133.1, 79.6)
- moved R513 9.35 mm to (140.1, 80.5)
- moved R514 9.35 mm to (140.1, 79.0), turned to 0 degrees
- moved R515 9.35 mm to (140.1, 77.5)
- moved R506 9.35 mm to (133.1, 74.8)
- moved C508 9.07 mm to (140.1, 89.4), turned to 0 degrees
- moved R508 8.79 mm to (134.1, 89.3), turned to 0 degrees
- moved C502 8.28 mm to (134.1, 77.2), turned to 180 degrees
- moved C504 6.87 mm to (129.2, 86.6)
- moved RN501 6.84 mm to (133.9, 85.7), turned to 0 degrees
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- renumbered C512 to C509, C513 to C510, C514 to C511, C515 to C512, R501 to R502, R502 to R503, R503 to R504, R504 to R505, R511 to R512, R512 to R513, R513 to R514, R514 to R515, R515 to R516, U504 to U503, U503 to U504
Connections:
- net /Current/HMSR_VOUT renamed /Current/VOUT
- C409 pad 1: +1.65V -> VDD
- C411 pad 1: +1.65V -> VDD
- R406 pad 2: /MCU/VOUTP -> Net-(U401--IN1)
- R507 pad 2: Net-(U505-+) -> Net-(U502A-+)
- R508 pad 1: Net-(U505--) -> +2V5
- R508 pad 2: Net-(R508-Pad2) -> Net-(U502B-+)
- R512 pad 1: Net-(U507-+) -> Net-(U502A--)
- R515 pad 2: GND -> VDD
- RN501 pad 1: Net-(R505-Pad2) -> Net-(R507-Pad1)
- RN501 pad 3: Net-(U506-+) -> Net-(U502A-+)
- RN502 pad 1: Net-(R508-Pad2) -> +2V5
- RN502 pad 3: Net-(U507-+) -> Net-(U502B-+)
- U401 pad 1: /MCU/VOUTP -> Net-(U401--IN1)
- U401 pad 2: +1.65V -> VDD
- U401 pad 4: /MCU/VOUTP -> Net-(U401--IN1)
- U401 pad 5: /MCU/VOUTN -> Net-(U401-OUT2)
- U402 pad 1: +1.65V -> unconnected-(U402-Vbias-Pad1)
- U403 pad 28: unconnected-(U403-PA4-Pad28) -> /Current/MCU_G100
- U403 pad 29: unconnected-(U403-PA5-Pad29) -> /Current/MCU_G10
- U403 pad 35: unconnected-(U403-PB1-Pad35) -> /Current/MCU_ZOFFS
- U403 pad 36: unconnected-(U403-PB2-Pad36) -> /Current/MCU_G1
- U403 pad 37: /Current/MCU_G100 -> unconnected-(U403-PE7-Pad37)
- U403 pad 38: /Current/MCU_G10 -> unconnected-(U403-PE8-Pad38)
- U403 pad 39: /Current/MCU_MEAS_ENA -> unconnected-(U403-PE9-Pad39)
- U403 pad 40: /Current/MCU_G1 -> unconnected-(U403-PE10-Pad40)
- U403 pad 41: /Current/MCU_DIV10 -> unconnected-(U403-PE11-Pad41)
- U403 pad 42: /Current/MCU_DIV100 -> unconnected-(U403-PE12-Pad42)
- U403 pad 43: /Current/MCU_ZOFFS -> unconnected-(U403-PE13-Pad43)
- U403 pad 44: /Current/MCU_DIV_ENA -> unconnected-(U403-PE14-Pad44)
- U403 pad 45: /Current/MCU_DIV1 -> unconnected-(U403-PE15-Pad45)
- U502 pad 1: /Current/MCU_DIV1 -> Net-(U502A--)
- U502 pad 10: +3.3VADC -> Net-(U502A--)
- U502 pad 11: Net-(R505-Pad2) -> GND
- U502 pad 12: +3.3V -> GND
- U502 pad 13: +5VL -> Net-(U502D--)
- U502 pad 14: Net-(U507-+) -> Net-(U502D--)
- U502 pad 15: Net-(U506--) -> (no net)
- U502 pad 16: /Current/MCU_DIV_ENA -> (no net)
- U502 pad 2: +3.3VADC -> Net-(U502A--)
- U502 pad 3: Net-(U506-+) -> Net-(U502A-+)
- U502 pad 4: GND -> +3.3V
- U502 pad 5: GND -> Net-(U502B-+)
- U502 pad 6: +3.3VADC -> VDD
- U502 pad 7: Net-(R505-Pad1) -> VDD
- U502 pad 8: /Current/MCU_DIV100 -> Net-(D501-K-Pad3)
- U502 pad 9: /Current/MCU_DIV10 -> Net-(U502C--)
- U503 pad 10: Net-(U507--) -> Net-(U502C--)
- U503 pad 14: Net-(R508-Pad2) -> Net-(U503-Pad14)
- U503 pad 15: Net-(U505--) -> Net-(U503-Pad14)
- U503 pad 16: /Current/MCU_MEAS_ENA -> Net-(R501-Pad1)
- U503 pad 2: Net-(U507--) -> Net-(U502C--)
- U503 pad 6: Net-(U507--) -> Net-(U502C--)
Routing:
- net VDD: track 0.00 -> 41.4 mm, vias 0 -> 3
- net +3.3VADC: track 49.2 -> 16.9 mm, vias 3 -> 2
- net /Current/MCU_MEAS_ENA: track 26.3 -> 0.00 mm, vias 2 -> 0
- net Net-(U507-+): track 24.5 -> 0.00 mm, vias 1 -> 0
- net Net-(R508-Pad2): track 22.9 -> 0.00 mm, vias 1 -> 0
- net /Current/MCU_DIV1: track 20.8 -> 0.00 mm, vias 2 -> 0
- net Net-(U505--): track 19.8 -> 0.00 mm, vias 1 -> 0
- net /Current/MCU_G100: track 23.8 -> 3.97 mm, vias 2 -> 0
- net /MCU/VOUTP: track 22.0 -> 2.61 mm
- net Net-(U507--): track 18.6 -> 0.00 mm
- net /Current/MCU_DIV_ENA: track 18.3 -> 0.00 mm, vias 2 -> 0
- net Net-(U502A--): track 0.00 -> 17.9 mm, vias 0 -> 2
- net Net-(U502A-+): track 0.00 -> 15.0 mm, vias 0 -> 1
- net Net-(U502C--): track 0.00 -> 14.8 mm
- net /Current/MCU_G1: track 25.4 -> 10.8 mm
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
Commit message: Development
Parts:
- added REF**: Symbol_Attention_Triangle_8x7mm_Copper, Symbol:Symbol_Attention_Triangle_8x7mm_Copper, F.Cu at (112.9, 64.8)
- added REF**: Symbol_Attention_Triangle_8x7mm_Copper, Symbol:Symbol_Attention_Triangle_8x7mm_Copper, B.Cu at (112.9, 64.8)
