File: HARDWARE/ETH1HMSR-SMS/ETH1HMSR-SMS.kicad_pcb (KiCad board)
At the start: 4 copper layers, 100 x 45 mm, 127 parts, among them J201 1715721, J301 RJ45_Wuerth_7499010121A, J401 20021111-00010T4LF, J501 1710072, Q201 SI5618A, Q202 MMBT3904, U201 TSR_1-2450, U202 LM1117MP-3.3/NOPB, U301 LAN8742A, U401 LT6350xMS8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

Commit message: Small improvements.
Parts:
- moved FID102 40.2 mm to (180.3, 63.5)
- moved FID104 40.2 mm to (180.3, 63.5)
- moved FID101 39.7 mm to (111.1, 101.9)
- moved FID103 39.7 mm to (111.1, 101.9)
