File: HARDWARE/ETH1HMSR-SMS/Current.kicad_sch (KiCad schematic)
At the start: 28 parts, among them J501 1710072, U501 HMSR-SMS, U502 DG419LDY, U503 DG411LEDQ, U504 OPA341UA, U505 OPA341UA

Commit message: SW and HW development
Parts:
- removed U503: DG411LEDQ, Package_SO:TSSOP-16_4.4x5mm_P0.65mm, symbol Analog_Switch:DG411xUE
- added C509, C510, C511, C512, C513, C514: 0.1u, Capacitor_SMD:C_0603_1608Metric_Pad1.08x0.95mm_HandSolder, symbol Device:C
- added C515: 100p, Capacitor_SMD:C_0603_1608Metric_Pad1.08x0.95mm_HandSolder, symbol Device:C
- added R513: RT1206BRE07900KL, Resistor_SMD:R_1206_3216Metric_Pad1.30x1.75mm_HandSolder, symbol Device:R
- added R514: 0, Resistor_SMD:R_0603_1608Metric_Pad0.98x0.95mm_HandSolder, symbol Device:R
- added R515: 100, Resistor_SMD:R_0603_1608Metric_Pad0.98x0.95mm_HandSolder, symbol Device:R
- added RN501: SOT-DIV23LF-03-9002-1002-DD, Package_TO_SOT_SMD:SOT-23, symbol Device:VoltageDivider_CenterPin3
- added U503, U506: DG412LEDQ, Package_SO:TSSOP-16_4.4x5mm_P0.65mm, symbol Analog_Switch:DG412xUE
- added U507: OPA341UA, Package_SO:SOIC-8_3.9x4.9mm_P1.27mm, symbol Amplifier_Operational:OPA340UA
- R507: value 10k -> 0
Connections:
- net +2V5: now also U506.10, U506.2, U506.6
- net +3.3V: now also C509.1, C510.1, U503.12 (VL), U506.12 (VL), U507.7 (V+)
- net +5VL: now also C511.1, C512.1, C513.1, C514.1, U503.13 (V+), U506.13 (V+); no longer R507.2
- net GND: now also C509.2, C510.2, C511.2, C512.2, C513.2, C514.2, C515.2, RN501.2, U503.4 (V-), U503.5 (GND), U506.4 (V-), U506.5 (GND), U507.4 (V-)
- net HMSR_VOUT: now also C515.1, R515.2; no longer D501.3 (K), R510.1, U505.6
- net MCU_G1: now also U503.1
- net MCU_G10: now also U503.8
- net MCU_G100: now also U503.9
- net at R510.2, R511.1: now also U503.7
- net at R511.2, R512.1: now also U503.11
- net at U505.2 (-): now also U503.10, U503.2, U503.6
- net at R508.2, R509.2, U505.3 (+): now also R514.1
- net at R507.1: now also U504.2 (-), U504.6, U503.15
- new net: D501.3 (K), R510.1, R514.2, R515.1, U503.3, U505.6
- new net: U506.15, U507.2 (-), U507.6
- new net: RN501.3, U506.3, U507.3 (+)
- new net: R507.2, R508.1, U503.14, U506.14
- new net: R513.1, U506.7
- new net: R513.2, RN501.1, U506.11
- new net MCU_DIV1: U506.1
- new net MCU_DIV10: U506.9
- new net MCU_DIV100: U506.8
- new net MCU_DIV_ENA: U506.16
- new net MCU_MEAS_ENA: U503.16
Other:
- moved on the sheet: C501, C502, C503, C504, C505, C506, C507, C508, D501, FB501, J501, R501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

Commit message: Development
Other:
- moved on the sheet: C501, C502, C503, C505, C507, C508, C509, C511, C513, C514, C515, D501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

Commit message: PCB
Parts:
- U502: value DG419LDY -> DG419LEDY
Changed lines of the file:
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@@
 			)
 		)
-		(property "Value" "DG419LDY"
+		(property "Value" "DG419LEDY"
 			(at 109.22 180.34 0)
 			(effects
@@
 			)
 		)
-		(property "Value" "DG419LDY"
+		(property "Value" "DG419LEDY"
 			(at 132.08 63.5 0)
 			(effects

Commit message: Development
Parts:
- removed R508: 2k/0.1%, Resistor_SMD:R_0603_1608Metric_Pad0.98x0.95mm_HandSolder, symbol Device:R
- removed R509: 4k/0.1%, Resistor_SMD:R_0603_1608Metric_Pad0.98x0.95mm_HandSolder, symbol Device:R
- added RN502: MPMT10012001AT1, Package_TO_SOT_SMD:SOT-23, symbol Device:VoltageDivider_CenterPin3
- renumbered C511 to C501, C503 to C502, C501 to C503, C512 to C504, C504 to C505, C502 to C506, C513 to C507, C505 to C508, C514 to C509, C509 to C510, C510 to C511, C506 to C512, C507 to C513, C508 to C514, R504 to R501, R501 to R502, R502 to R503, R503 to R504, R513 to R505, R505 to R506, R506 to R507, R507 to R508, R514 to R511, R510 to R512, R511 to R513, R512 to R514, U506 to U502, U502 to U503, U503 to U504, U504 to U505, U507 to U506, U505 to U507
Connections:
- net +2V5: no longer R502.1, U502.10, U502.2, U502.6
- net +5VL: now also R502.1
- net GND: now also RN502.2
- net at R511.1, U507.3 (+): now also U502.14, RN502.3
- net at R508.2, U504.14: now also RN502.1; no longer U502.14
- new net +3.3VADC: U502.10, U502.2, U502.6
Other:
- moved on the sheet: C501, C502, C503, C504, C505, C506, C507, C508, C509, C510, C511, C512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

Commit message: Development
Parts:
- removed C509, C510, C511: 0.1u, Capacitor_SMD:C_0603_1608Metric_Pad1.08x0.95mm_HandSolder, symbol Device:C
- removed R505: RT1206BRE07900KL, Resistor_SMD:R_1206_3216Metric_Pad1.30x1.75mm_HandSolder, symbol Device:R
- removed U502: DG412LEDQ, Package_SO:TSSOP-16_4.4x5mm_P0.65mm, symbol Analog_Switch:DG412xUE
- removed U505, U506, U507: OPA341UA, Package_SO:SOIC-8_3.9x4.9mm_P1.27mm, symbol Amplifier_Operational:OPA340UA
- added R501: 100k, Resistor_SMD:R_0603_1608Metric_Pad0.98x0.95mm_HandSolder, symbol Device:R
- added R509, R510: 2k5/0.1%, Resistor_SMD:R_0603_1608Metric_Pad0.98x0.95mm_HandSolder, symbol Device:R
- added R511: 100k/0.1%, Resistor_SMD:R_0603_1608Metric_Pad0.98x0.95mm_HandSolder, symbol Device:R
- added U502: OPA4340UA, Package_SO:SSOP-16_3.9x4.9mm_P0.635mm, symbol Amplifier_Operational:OPA4340UA
- R507: value 1k -> 1k/0.1%
- R508: value 0 -> 1k/0.1%
- RN501: value SOT-DIV23LF-03-9002-1002-DD -> MPMT10012001AT1
- renumbered C512 to C509, C513 to C510, C514 to C511, C515 to C512, R501 to R502, R502 to R503, R503 to R504, R504 to R505, R511 to R512, R512 to R513, R513 to R514, R514 to R515, R515 to R516, U504 to U503, U503 to U504
Connections:
- net +2V5: now also R508.1, RN502.1
- net +3.3V: now also R501.2, U502.4 (V+)
- net GND: now also R509.2, R510.2, U502.11 (V-), U502.12 (+); no longer R515.2
- net at U503.10, U503.2, U503.6: now also U502.9 (-)
- net at R512.1: now also R511.1, U502.1, U502.10 (+), U502.2 (-); no longer RN502.3
- net at D501.3 (K), R512.2, R513.1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: now also U502.8
- net at RN501.3: now also R507.2, R509.1, U502.3 (+)
- net at RN501.1: now also R507.1, U504.1
- net at U503.15: now also U503.14; no longer R508.1
- net HMSR_VOUT renamed VOUT
- net MCU_MEAS_ENA: no longer names the net of U503.16
- net MCU_MEAS_ENA: now also R501.1
- new net: U502.13 (-), U502.14
- new net: R508.2, R510.1, RN502.3, U502.5 (+)
- new net VDD: R511.2, R515.2, U502.6 (-), U502.7
Other:
- moved on the sheet: C501, C502, C503, C504, C505, C506, C507, C508, C509, C510, C511, C512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

Commit message: Development
Other:
- moved on the sheet: U502E, U503E, U504B

Commit message: development
Parts:
- C512: value 100p -> DNP; now not fitted
- D501: value BAV99 -> BAV199
- R507, R508, R509, R510: now not fitted
- R512: value 0 -> DNP; now not fitted
- R516: value 100 -> 0
Changed lines of the file:
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@@
 		(in_bom yes)
 		(on_board yes)
-		(dnp no)
+		(dnp yes)
 		(fields_autoplaced yes)
 		(property "Reference" "C512"
-			(at 267.335 70.485 0)
+			(at 267.97 69.8499 0)
 			(effects
 				(font
@@
 			)
 		)
-		(property "Value" "100p"
-			(at 267.335 73.025 0)
+		(property "Value" "DNP"
+			(at 267.97 72.3899 0)
 			(effects
 				(font
@@
 		(in_bom yes)
 		(on_board yes)
-		(dnp no)
+		(dnp yes)
 		(fields_autoplaced yes)
 		(property "Reference" "R509"
@@
 			)
 		)
-		(property "Value" "100"
+		(property "Value" "0"
 			(at 259.08 64.77 90)
 			(effects
@@
 		(in_bom yes)
 		(on_board yes)
-		(dnp no)
+		(dnp yes)
 		(fields_autoplaced yes)
 		(property "Reference" "R512"
@@
 			)
 		)
-		(property "Value" "0"
+		(property "Value" "DNP"
 			(at 229.87 49.53 90)
 			(effects
@@
 		(in_bom yes)
 		(on_board yes)
-		(dnp no)
+		(dnp yes)
 		(property "Reference" "R507"
 			(at 161.29 57.658 90)
@@
 		(in_bom yes)
 		(on_board yes)
-		(dnp no)
+		(dnp yes)
 		(fields_autoplaced yes)
 		(property "Reference" "R510"
@@
 		(in_bom yes)
 		(on_board yes)
-		(dnp no)
+		(dnp yes)
 		(property "Reference" "R508"
 			(at 161.29 100.076 90)
@@
 			)
 		)
-		(property "Value" "BAV99"
+		(property "Value" "BAV199"
 			(at 247.65 70.485 90)
 			(effects
