File: HARDWARE/ETH1HMSR-SMS/Current.kicad_sch (KiCad schematic)
At the start: 38 parts, among them J501 1710072, U501 HMSR-SMS, U502 OPA4340EA, U503 DG412LEDQ, U504 DG419LEDY

Commit message: BOM updated
Parts:
- D501: now not fitted; now left out of the parts list
Changed lines of the file:
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@@
 		(unit 1)
 		(exclude_from_sim no)
-		(in_bom yes)
+		(in_bom no)
 		(on_board yes)
-		(dnp no)
+		(dnp yes)
 		(property "Reference" "D501"
 			(at 245.11 64.77 90)
