File: HARDWARE/ETH1HMSR-SMS/MCU.kicad_sch (KiCad schematic)
At the start: 40 parts, among them J401 20021111-00010T4LF, U401 LT6350xMS8, U402 REF2033AIDDCT, U403 STM32H743VITx, U404 24LC08B-E/MS, Y401 NX5032GA-16

Commit message: BOM updated
Parts:
- C413, R408: now left out of the parts list
Changed lines of the file:
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@@
 		(unit 1)
 		(exclude_from_sim no)
-		(in_bom yes)
+		(in_bom no)
 		(on_board yes)
 		(dnp yes)
@@
 		(unit 1)
 		(exclude_from_sim no)
-		(in_bom yes)
+		(in_bom no)
 		(on_board yes)
 		(dnp yes)
